File: Guitar_Electronics/CV_Pot/CV_Pot.sch (EAGLE design)
At the start: 6 parts

Commit message: Licenses
Parts:
- added C2: 10uF, resistor:C-EUC0805
- added SJ1: (no value), jumper:SJ
Connections:
- net GND: now also C2.2
- net N$1: now also C2.1, SJ1.2
- net N$2: now also SJ1.1
Other:
- note added: "CV_Pot for Nexus Project by Cycfi Research is licensed under a Creative Commons Attribution-ShareAlike 4.0 International License. Copyright CYCFI Research Inc. 2013-2016"
- note removed: "Nexus Project by Cycfi Research is licensed under a Creative Commons Attribution-NonCommercial 4.0 International License. http://creativecommons.org/licenses/by-nc/4.0/ Copyright CYCFI Research Inc. 2013-2016"
Changed lines of the file:
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@@
 <part name="C1" library="resistor" deviceset="C-EU" device="C0603" value="0.1uF"/>
 <part name="R1" library="resistor" deviceset="R-EU_" device="R0402" value="20K"/>
+<part name="SJ1" library="jumper" deviceset="SJ" device=""/>
+<part name="C2" library="resistor" deviceset="C-EU" device="C0805" value="10uF"/>
 </parts>
 <sheets>
@@
 <text x="149.225" y="118.11" size="1.778" layer="95">OUT</text>
 <text x="237.49" y="6.985" size="2.1844" layer="95">v0.96</text>
-<text x="10.16" y="7.62" size="2.54" layer="95">Nexus Project by Cycfi Research is licensed under a
-Creative Commons Attribution-NonCommercial 4.0
-International License.
-http://creativecommons.org/licenses/by-nc/4.0/
+<text x="10.16" y="7.62" size="2.54" layer="95">CV_Pot for Nexus Project by Cycfi Research is licensed under a
+Creative Commons Attribution-ShareAlike 4.0 International License.
 Copyright CYCFI Research Inc. 2013-2016</text>
 </plain>
@@
 <attribute name="VALUE" x="88.392" y="78.867" size="1.778" layer="96" rot="R90"/>
 </instance>
-<instance part="GND2" gate="1" x="90.805" y="80.01" smashed="yes" rot="R90">
-<attribute name="VALUE" x="94.107" y="78.867" size="1.778" layer="96" rot="R90"/>
+<instance part="GND2" gate="1" x="90.17" y="80.01" smashed="yes" rot="R90">
+<attribute name="VALUE" x="93.472" y="78.867" size="1.778" layer="96" rot="R90"/>
 </instance>
 <instance part="POT1" gate="G$1" x="121.92" y="97.155" smashed="yes">
@@
 <attribute name="NAME" x="124.46" y="114.3" size="1.778" layer="95"/>
 <attribute name="VALUE" x="124.46" y="111.76" size="1.778" layer="96"/>
+</instance>
+<instance part="SJ1" gate="1" x="111.76" y="113.03" rot="R90"/>
+<instance part="C2" gate="G$1" x="90.17" y="115.57" smashed="yes">
+<attribute name="NAME" x="94.234" y="115.951" size="1.778" layer="95"/>
+<attribute name="VALUE" x="94.234" y="113.411" size="1.778" layer="96"/>
 </instance>
 </instances>
@@
 <wire x1="139.7" y1="123.19" x2="121.92" y2="123.19" width="0.1524" layer="91"/>
 <wire x1="121.92" y1="123.19" x2="121.92" y2="118.11" width="0.1524" layer="91"/>
+<pinref part="SJ1" gate="1" pin="2"/>
+<wire x1="111.76" y1="118.11" x2="121.92" y2="118.11" width="0.1524" layer="91"/>
+<junction x="121.92" y="118.11"/>
+<pinref part="C2" gate="G$1" pin="1"/>
+<wire x1="121.92" y1="123.19" x2="90.17" y2="123.19" width="0.1524" layer="91"/>
+<wire x1="90.17" y1="123.19" x2="90.17" y2="118.11" width="0.1524" layer="91"/>
+<junction x="121.92" y="123.19"/>
 </segment>
 </net>
@@
 <pinref part="POT1" gate="G$1" pin="3"/>
 <wire x1="121.92" y1="107.95" x2="121.92" y2="102.235" width="0.1524" layer="91"/>
+<pinref part="SJ1" gate="1" pin="1"/>
+<wire x1="111.76" y1="107.95" x2="121.92" y2="107.95" width="0.1524" layer="91"/>
+<junction x="121.92" y="107.95"/>
 </segment>
 </net>
@@
 <wire x1="97.155" y1="89.535" x2="97.155" y2="120.65" width="0.1524" layer="91"/>
 <pinref part="GND2" gate="1" pin="P"/>
-<wire x1="90.805" y1="82.55" x2="90.805" y2="89.535" width="0.1524" layer="91"/>
-<wire x1="90.805" y1="89.535" x2="97.155" y2="89.535" width="0.1524" layer="91"/>
+<wire x1="90.17" y1="82.55" x2="90.17" y2="89.535" width="0.1524" layer="91"/>
+<wire x1="90.17" y1="89.535" x2="97.155" y2="89.535" width="0.1524" layer="91"/>
 <pinref part="GND1" gate="1" pin="P"/>
 <wire x1="85.09" y1="82.55" x2="85.09" y2="89.535" width="0.1524" layer="91"/>
-<wire x1="85.09" y1="89.535" x2="90.805" y2="89.535" width="0.1524" layer="91"/>
-<junction x="90.805" y="89.535"/>
+<wire x1="85.09" y1="89.535" x2="90.17" y2="89.535" width="0.1524" layer="91"/>
+<junction x="90.17" y="89.535"/>
 <junction x="97.155" y="89.535"/>
 <wire x1="139.7" y1="120.65" x2="97.155" y2="120.65" width="0.1524" layer="91"/>
+<pinref part="C2" gate="G$1" pin="2"/>
+<wire x1="90.17" y1="110.49" x2="90.17" y2="89.535" width="0.1524" layer="91"/>
 </segment>
 </net>
