File: Guitar_Electronics/CV_Pot/CV_Pot.brd (EAGLE design)
At the start: 17 x 24 mm, 6 parts

Commit message: Licenses
Parts:
- added C2: 10uF, resistor:C0805
- added SJ1: (no value), jumper:SJ
Connections:
- net GND: now also C2.2
- net N$1: now also C2.1, SJ1.2
- net N$2: now also SJ1.1
Routing:
- net GND: track 47.6 -> 64.9 mm, vias 2 -> 3
- net N$1: track 7.53 -> 21.1 mm, vias 0 -> 2
- net N$2: track 15.8 -> 22.9 mm
Changed lines of the file:
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@@
 <setting verticaltext="up"/>
 </settings>
-<grid distance="1" unitdist="mm" unit="mm" style="lines" multiple="1" display="yes" altdistance="0.025" altunitdist="inch" altunit="inch"/>
+<grid distance="0.25" unitdist="mm" unit="mm" style="lines" multiple="1" display="yes" altdistance="0.025" altunitdist="inch" altunit="inch"/>
 <layers>
 <layer number="1" name="Top" color="4" fill="1" visible="yes" active="yes"/>
@@
 <layer number="220" name="220bmp" color="21" fill="1" visible="no" active="no"/>
 <layer number="221" name="221bmp" color="22" fill="1" visible="no" active="no"/>
-<layer number="222" name="222bmp" color="23" fill="1" visible="no" active="no"/>
 <layer number="223" name="223bmp" color="24" fill="1" visible="no" active="no"/>
 <layer number="224" name="224bmp" color="25" fill="1" visible="no" active="no"/>
@@
 <board>
 <plain>
-<circle x="8.49" y="15.25" radius="8.5" width="0.254" layer="21"/>
+<circle x="8.49" y="15.25" radius="8.5" width="0.254" layer="25"/>
 <wire x1="17" y1="3" x2="17" y2="19.5" width="0.15" layer="20"/>
 <wire x1="17" y1="19.5" x2="12.5" y2="24" width="0.15" layer="20" curve="90"/>
@@
 <wire x1="3" y1="0" x2="14" y2="0" width="0.15" layer="20"/>
 <wire x1="14" y1="0" x2="17" y2="3" width="0.15" layer="20" curve="90"/>
-<text x="14.099996875" y="20.500009375" size="0.8128" layer="126" rot="MR0">C1</text>
-<text x="15.79999375" y="20.500009375" size="0.8128" layer="126" rot="MR0">R1</text>
-<text x="11.5" y="22" size="1.016" layer="126" ratio="10" rot="SMR0">CV POT</text>
-<text x="6.3" y="20.9" size="0.8128" layer="126" ratio="10" rot="MR0">OUT</text>
-<text x="8.8" y="20.9" size="0.8128" layer="126" ratio="10" rot="MR0">-</text>
-<text x="11.4" y="20.85" size="0.8128" layer="126" ratio="10" rot="MR0">+</text>
+<text x="14.099996875" y="20.500009375" size="0.8128" layer="26" rot="MR0">C1</text>
+<text x="15.79999375" y="20.500009375" size="0.8128" layer="26" rot="MR0">R1</text>
+<text x="11.5" y="22" size="0.8128" layer="26" ratio="10" rot="SMR0">CV POT</text>
+<text x="6.3" y="20.9" size="0.8128" layer="26" ratio="10" rot="MR0">OUT</text>
+<text x="8.8" y="20.9" size="0.8128" layer="26" ratio="10" rot="MR0">-</text>
+<text x="11.4" y="20.85" size="0.8128" layer="26" ratio="10" rot="MR0">+</text>
 <wire x1="17" y1="3" x2="17" y2="19.5" width="0.15" layer="125"/>
 <wire x1="17" y1="19.5" x2="12.5" y2="24" width="0.15" layer="125" curve="90"/>
@@
 </element>
 <element name="R1" library="resistor" package="R0402" value="20K" x="15" y="18.8" smashed="yes" rot="MR90">
-<attribute name="VALUE" x="12.968" y="18.165" size="1.27" layer="28" rot="MR90"/>
+<attribute name="VALUE" x="12.968" y="18.165" size="0.8128" layer="28" rot="MR90"/>
+</element>
+<element name="SJ1" library="jumper" package="SJ" value="" x="13.75" y="9.75" smashed="yes" rot="MR90">
+<attribute name="VALUE" x="13.75" y="10.1501" size="0.02" layer="28" rot="MR90"/>
+</element>
+<element name="C2" library="resistor" package="C0805" value="10uF" x="14" y="13.75" smashed="yes" rot="MR90">
+<attribute name="NAME" x="16.139" y="13.512" size="0.8128" layer="26" rot="MR0"/>
+<attribute name="VALUE" x="11.968" y="12.861" size="0.8128" layer="28" rot="MR90"/>
 </element>
 </elements>
@@
 <via x="2.5" y="17.5" extent="1-16" drill="0.4"/>
 <wire x1="2.5" y1="17.5" x2="2.5" y2="21" width="0.4064" layer="1"/>
+<contactref element="C2" pad="2"/>
+<wire x1="3.49" y1="2.97" x2="3.49" y2="3.24" width="0.4064" layer="1"/>
+<wire x1="3.49" y1="3.24" x2="10.75" y2="10.5" width="0.4064" layer="1"/>
+<wire x1="10.75" y1="10.5" x2="10.75" y2="13.5" width="0.4064" layer="1"/>
+<wire x1="10.75" y1="13.5" x2="11.5" y2="14.25" width="0.4064" layer="1"/>
+<via x="11.5" y="14.25" extent="1-16" drill="0.4"/>
+<wire x1="11.5" y1="14.25" x2="12.9" y2="14.25" width="0.4064" layer="16"/>
+<wire x1="14" y1="14.6" x2="13.25" y2="14.6" width="0.4064" layer="16"/>
+<wire x1="13.25" y1="14.6" x2="12.9" y2="14.25" width="0.4064" layer="16"/>
 </signal>
 <signal name="N$1">
@@
 <wire x1="14.5" y1="21.3" x2="15" y2="20.8" width="0.6096" layer="16"/>
 <wire x1="15" y1="20.8" x2="15" y2="19.45" width="0.6096" layer="16"/>
+<contactref element="SJ1" pad="2"/>
+<contactref element="C2" pad="1"/>
+<wire x1="11.04" y1="18.9" x2="11.04" y2="17.79" width="0.4064" layer="16"/>
+<wire x1="11.04" y1="17.79" x2="11" y2="17.75" width="0.4064" layer="16"/>
+<via x="11" y="17.75" extent="1-16" drill="0.4"/>
+<wire x1="11" y1="17.75" x2="11" y2="17.25" width="0.4064" layer="1"/>
+<wire x1="11" y1="17.25" x2="11.75" y2="16.5" width="0.4064" layer="1"/>
+<wire x1="11.75" y1="16.5" x2="12.75" y2="16.5" width="0.4064" layer="1"/>
+<wire x1="12.75" y1="16.5" x2="13.25" y2="16" width="0.4064" layer="1"/>
+<wire x1="13.25" y1="16" x2="13.25" y2="13.25" width="0.4064" layer="1"/>
+<wire x1="13.25" y1="13.25" x2="12" y2="12" width="0.4064" layer="1"/>
+<via x="12" y="12" extent="1-16" drill="0.4"/>
+<wire x1="12" y1="12" x2="12.35" y2="12" width="0.4064" layer="16"/>
+<wire x1="12.35" y1="11.662" x2="12.6" y2="11.662" width="0.8128" layer="16"/>
+<wire x1="12.6" y1="11.662" x2="13.75" y2="10.512" width="0.8128" layer="16"/>
+<wire x1="14" y1="12.9" x2="12.9" y2="12.9" width="0.4064" layer="16"/>
+<wire x1="12.9" y1="12.9" x2="12" y2="12" width="0.4064" layer="16"/>
+<wire x1="12.35" y1="12" x2="12.35" y2="11.662" width="0" layer="19" extent="16-16"/>
 </signal>
 <signal name="N$2">
@@
 <contactref element="POT1" pad="A3"/>
 <wire x1="13.49" y1="2.97" x2="13.49" y2="2.99" width="0.6096" layer="16"/>
-<wire x1="13.49" y1="2.99" x2="14.8" y2="4.3" width="0.6096" layer="16"/>
-<wire x1="14.8" y1="4.3" x2="14.8" y2="17.95" width="0.6096" layer="16"/>
 <wire x1="14.8" y1="17.95" x2="15" y2="18.15" width="0.6096" layer="16"/>
+<contactref element="SJ1" pad="1"/>
+<wire x1="14.8" y1="17.95" x2="15.05" y2="17.95" width="0.8128" layer="16"/>
+<wire x1="15.05" y1="17.95" x2="15.75" y2="17.25" width="0.8128" layer="16"/>
+<wire x1="15.75" y1="17.25" x2="15.75" y2="5.23" width="0.8128" layer="16"/>
+<wire x1="15.75" y1="5.23" x2="13.49" y2="2.97" width="0.8128" layer="16"/>
+<wire x1="13.75" y1="8.988" x2="13.75" y2="3.23" width="0.8128" layer="16"/>
+<wire x1="13.75" y1="3.23" x2="13.49" y2="2.97" width="0.8128" layer="16"/>
 </signal>
 <signal name="OUT">

Commit message: Change 10uF to 1uF in the schematics and BOM file
Parts:
- C2: value 10uF -> 1uF
Changed lines of the file:
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@@
 <attribute name="VALUE" x="13.75" y="10.1501" size="0.02" layer="28" rot="MR90"/>
 </element>
-<element name="C2" library="resistor" package="C0805" value="10uF" x="14" y="13.75" smashed="yes" rot="MR90">
+<element name="C2" library="resistor" package="C0805" value="1uF" x="14" y="13.75" smashed="yes" rot="MR90">
 <attribute name="NAME" x="16.139" y="13.512" size="0.8128" layer="26" rot="MR0"/>
 <attribute name="VALUE" x="11.968" y="12.861" size="0.8128" layer="28" rot="MR90"/>
