File: Guitar_Electronics/19P_Lemo_Connector/2mm_Header_Adaptor/2mm_Header_Adaptor.sch (EAGLE design)
At the start: 8 parts

Commit message: *Edit Logo *Check BOM *Added 19P Connector Files
Parts:
- removed C1: 0.1uF, resistor:C-EUC0603
- removed C2: 10uF, resistor:C-EUC0805
- removed GND1, GND2: (no value), wirepad:SMD2
- removed POT1: 25K, CYCFI_Passive:POTPDB181GTR
- removed R1: 20K, resistor:R-EU_R0402
- removed SJ1: (no value), jumper:SJ
- added H2, H3: 7P_ZIF_59453-071110EDHLF, CYCFI_Con:7P_ZIF_59453-071110EDHLF
- added H4: 2X10, headers(2mm):2X10
- H1: value 3PIN-SMD-2.54MM -> 7P_ZIF_59453-071110EDHLF; device CYCFI_Con:3PIN-SMD-2.54MM -> CYCFI_Con:7P_ZIF_59453-071110EDHLF
Connections:
- removed net N$1: C2.1, H1.3, R1.2, SJ1.2
- removed net N$2: POT1.3, R1.1, SJ1.1
- removed net OUT: C1.1, H1.1, POT1.2
- new net CH1: H1.7, H4.15
- new net CH10: H2.4, H4.8
- new net CH11: H2.3, H4.5
- new net CH12: H2.1, H4.6
- new net CH2: H1.6, H4.16
- new net CH3: H1.5, H4.13
- new net CH4: H1.4, H4.14
- new net CH5: H1.3, H4.11
- new net CH6: H1.1, H4.12
- new net CH7: H2.7, H4.9
- new net CH8: H2.6, H4.10
- new net CH9: H2.5, H4.7
- new net MIDI1: H3.7, H4.3
- new net MIDI2: H3.6, H4.4
- new net MIDI3: H3.5, H4.1
- new net NC1: H4.17
- new net NC2: H4.18
- new net VCC: H3.1, H3.3, H4.2
- new net VGND: H3.4, H4.19
- net GND: now also H2.2, H3.2, H4.20; no longer C1.2, C2.2, GND1.P, GND2.P, POT1.1
Other:
- note added: "1x7 FPC Connector"
- note added: "2mm Adaptor"
- note added: "2mm Adaptor for Nexus Project by Cycfi Research is licensed under a Creative Commons Attribution-ShareAlike 4.0 International License. Copyright CYCFI Research Inc. 2013-2016"
- note added: "CH1"
- note added: "CH10"
- note added: "CH11"
- note added: "CH12"
- note added: "CH13"
- note added: "CH14"
- note added: "CH15"
- note added: "CH2"
- note added: "CH3"
- note added: "CH4"
- note added: "CH5"
- note added: "CH6"
- note added: "CH7"
- note added: "CH8"
- note added: "CH9"
- note added: "NC"
- note added: "SGND"
- note added: "VCC"
- note added: "v0.92"
- note removed: "CV_Pot for Nexus Project by Cycfi Research is licensed under a Creative Commons Attribution-ShareAlike 4.0 International License. Copyright CYCFI Research Inc. 2013-2016"
- note removed: "Control Voltage Pot - MIDI"
- note removed: "OUT"
- note removed: "VCC(9V)"
- note removed: "v0.96"
