File: guitar_electronics/cv_pot/cv_pot.brd (EAGLE design)
At the start: 17 x 24 mm, 8 parts

Commit message: commit and push eagle files for Nexus v2.3
Parts:
- removed R1: 20K, resistor:R0402
- removed SJ1: (no value), jumper:SJ
- added C3: 1uF, resistor:C0603
- added U1: L78LXX, CYCFI_Power:SOT89
- C1: device resistor:C0603 -> resistor:C0402
- C2: device resistor:C0805 -> resistor:C0603
- moved C1 10.9 mm to (12.0, 8.00), turned to 180 degrees
- moved C2 5.62 mm to (12.0, 19.0), turned to 0 degrees
- moved H1 3.00 mm to (5.50, 19.0)
Connections:
- net GND: now also C2.1, C3.1, U1.2, U1.2@1; no longer C2.2
- net N$1: now also C2.2, U1.3; no longer C2.1, R1.2, SJ1.2
- net N$2: now also C3.2, U1.1; no longer R1.1, SJ1.1
Routing:
- net GND: track 64.9 -> 0.00 mm, vias 3 -> 0
- net N$1: track 21.1 -> 5.76 mm, vias 2 -> 0
- net N$2: track 22.9 -> 15.1 mm
- net OUT: track 26.8 -> 26.2 mm
Other:
- board text added: "CV POT v2.3"
- board text added: "GND"
- board text added: "V+"
- board text removed: "+"
- board text removed: "-"
- board text removed: "C1"
- board text removed: "CV POT"
- board text removed: "R1"
