File: guitar_electronics/cv_pot/cv_pot.sch (EAGLE design)
At the start: 8 parts

Commit message: commit and push eagle files for Nexus v2.3
Parts:
- removed R1: 20K, resistor:R-EU_R0402
- removed SJ1: (no value), jumper:SJ
- added C3: 1uF, resistor:C-EUC0603
- added U1: L78LXX, CYCFI_Power:L78LXX
- C1: device resistor:C-EUC0603 -> resistor:C-EUC0402
- C2: device resistor:C-EUC0805 -> resistor:C-EUC0603
Connections:
- net GND: now also C2.1, C3.1, U1.GND, U1.GND1; no longer C2.2
- net N$1: now also C2.2, U1.OUT; no longer C2.1, R1.2, SJ1.2
- net N$2: now also C3.2, U1.IN; no longer R1.1, SJ1.1
Other:
- note added: "CV_Pot for Nexus Project by Cycfi Research is licensed under a Creative Commons Attribution-ShareAlike 4.0 International License. Copyright CYCFI Research Inc. 2013-2020"
- note added: "VCC"
- note added: "v2.3"
- note removed: "2017030"
- note removed: "CV_Pot for Nexus Project by Cycfi Research is licensed under a Creative Commons Attribution-ShareAlike 4.0 International License. Copyright CYCFI Research Inc. 2013-2017"
- note removed: "VCC(9V)"
- note removed: "v0.96"
- moved on the sheet: C1, C2, H1, POT1
