File: guitar_electronics/cv_switch/cv_switch.sch (EAGLE design)
At the start: 8 parts

Commit message: commit and push eagle files for Nexus v2.3
Parts:
- added C3: 10uF, resistor:C-EUC0603
- added U1: CJ75L05, CYCFI_Power:L78LXX
- C1, C2: value 10uF -> 1uF; device resistor:C-EUC0805 -> resistor:C-EUC0603
- R1: value 4.7K -> 1.5K
- R2, R3: value 2.7K -> 3K
- R4: value 2K -> 1.5K
Connections:
- removed net N$2: R1.1, R2.2, U$1.N1
- new net +5V: C2.1, R1.2, R2.2, U1.IN
- new net N$7: R1.1, U$1.N1
- net GND: now also C3.2, U1.GND, U1.GND1
- net N$1: now also C1.1, U1.OUT; no longer C2.1, R1.2
- net OUT: now also C3.1; no longer C1.1
Other:
- note added: "1.25V"
- note added: "2.5V"
- note added: "5V"
- note added: "CJ75L05"
- note added: "CV Switch for Nexus Project by Cycfi Research is licensed under a Creative Commons Attribution-ShareAlike 4.0 International License. Copyright CYCFI Research Inc. 2013-2020"
- note added: "VCC"
- note added: "v2.3"
- note removed: "1.2V"
- note removed: "2.4V"
- note removed: "201031"
- note removed: "4.8V"
- note removed: "CV Switch for Nexus Project by Cycfi Research is licensed under a Creative Commons Attribution-ShareAlike 4.0 International License. Copyright CYCFI Research Inc. 2013-2017"
- note removed: "VCC(9V)"
- note removed: "v0.92"
- moved on the sheet: C1, C2, R1
