File: breakout_box/gk_+_midi_module/gk+midi board.sch (EAGLE design)
At the start: 114 parts, among them Q1 QUARZ5, T1 2N2222, T2 2N2222, U1 LMV324, U3 L78LXX, U4 MIC5205-3.3, U5 MSP430G2553RHB32, U7 TLV2170DGKT

Commit message: update boms and pdf for shematics files
Parts:
- removed C39, C40: 4.7uF, resistor:C-EUC0603
- removed C41, C42: 0.1uF, resistor:C-EUC0402
- removed C43: 0.01uF, resistor:C-EUC0402
- removed C44: 0.1uF, resistor:C-EUC0603
- removed H9: (no value), con-lstb:MA08-1
- removed R55, R56, R57: 10k, resistor:R-EU_R0402
- removed R74, R75: 1K, resistor:R-EU_R0402
- removed U7: TLV2170DGKT, CYCFI_semicon:TLV2170DGKT
- added C32: 10uf, resistor:C-EUC0805
- added C33: 2.2uf, resistor:C-EUC0805
- added C34: 0.1uf, resistor:C-EUC0603
- added C35: 1nF, resistor:C-EUC0402
- added C36, C37: 12pF, ssmd:C_SMD0603
- added H7: DNP, con-lstb:MA08-1
- added R20: 18K, resistor:R-EU_R0402
- added R21: 470K, resistor:R-EU_R0402
- added R22, R23: 100R, resistor:R-EU_R0402
- added R41: 47K, resistor:R-EU_R0402
- added U6: MSP430G2553RHB32, CYCFI_IC:MSP430G2553RHB32
- C1: value 10uF -> 100uF; device resistor:C-EUC0805 -> resistor:CPOL-EU153CLV-0505
- C11: value 0.1uF -> 10uF; device resistor:C-EUC0603 -> resistor:C-EUC0805
- C13: value 0.1uF -> 0.47uF
- C14: value 0.1uF -> 0.01uF; device resistor:C-EUC0603 -> resistor:C-EUC0402
- C15, C16: value 0.1uF -> 4.7uF
- C17: device resistor:C-EUC0603 -> resistor:C-EUC0402
- C18: value 1nF -> 0.1uF
- C19: value 1uF -> 0.1uF; device resistor:C-EUC0402 -> resistor:C-EUC0603
- C2: value 0.1uF -> 100uF; device resistor:C-EUC0603 -> resistor:CPOL-EU153CLV-0505
- C20: value 33uf -> 0.1uF; device resistor:C-EUC0805 -> resistor:C-EUC0603
- C21: value 10uf -> 0.1uF; device resistor:C-EUC0805 -> resistor:C-EUC0603
- C22: value 2.2uf -> 10uF
- C26: value 100uF -> 0.1uF; device resistor:CPOL-EU153CLV-0505 -> resistor:C-EUC0603
- C27: value 100uF -> 1uF; device resistor:CPOL-EU153CLV-0505 -> resistor:C-EUC0402
- C28: value 0.1uf -> 0.1uF
- C29: value 12pF -> 0.1uF; device ssmd:C_SMD0603 -> resistor:C-EUC0603
- C3, C7: value 10uF -> 0.1uF; device resistor:C-EUC0805 -> resistor:C-EUC0603
- C30: value 12pF -> 1uF; device ssmd:C_SMD0603 -> resistor:C-EUC0402
- C31: value 0.47uF -> 33uf; device resistor:C-EUC0603 -> resistor:C-EUC0805
- C9: value 1uF -> 10uF; device resistor:C-EUC0402 -> resistor:C-EUC0805
- H1, H2: value DNP -> (none)
- H3: value DNP -> (none); device con-lstb:MA04-2 -> con-lstb:MA08-1
- H5: value (none) -> DNP; device con-lstb:MA04-1 -> con-lstb:MA04-2
- H6: value (none) -> DNP
- H8: device con-lstb:MA08-1 -> con-lstb:MA04-1
- R1, R2: value 220R -> 100K; device resistor:R-EU_R0603 -> resistor:R-EU_R0402
- R10, R12, R8: value 5.1k -> 5k
- R11, R7, R9: value 10k -> 5k
- R13, R14, R15, R16, R17, R18: value 100K -> 5k
- R19: value 47K -> 10K
- R24: value 18K -> 5.1k
- R25: value 100R -> 5.1k
- R26: value 10K -> 5.1k
- R27: value 100R -> 10k
- R28: value 470K -> 10k
- R29, R35, R36, R37: value 5k -> 10k
- R3: value 1K -> 100K
- R30, R31: value 5k -> 220R; device resistor:R-EU_R0402 -> resistor:R-EU_R0603
- R32, R33, R34: value 5k -> 1K
- R38, R39, R40: value 5k -> 5.1k
- R4, R5, R6: value 5.1k -> 100K
- U1: value LMV324 -> (none); device CYCFI_semicon:LMV324 -> CYCFI_semicon:TLV2170DGKT
- U2: value (none) -> LMV324; device CYCFI_semicon:TLV2170DGKT -> CYCFI_semicon:LMV324
- U3: value L78LXX -> TLV2170DGKT; device CYCFI_Power:L78LXX -> CYCFI_semicon:TLV2170DGKT
- U4: value MIC5205-3.3 -> L78LXX; device v-reg-micrel:MIC5219BM5 -> CYCFI_Power:L78LXX
- U5: value MSP430G2553RHB32 -> MIC5205-3.3; device CYCFI_IC:MSP430G2553RHB32 -> v-reg-micrel:MIC5219BM5
- renumbered D3 to D2, D4 to D1, TP_10 to TP_2, TP_11 to TP_3, TP_12 to TP_4, TP_13 to TP_5, TP_14 to TP_6, TP_15 to TP_7, TP_9 to TP_1, U$3 to U$1
Connections:
- net !RST: now also C35.1, H8.2, R41.2, U6.RST; no longer C18.1, H5.2, R19.2, U5.RST
- net +3.3V: now also C31.1, C32.1, C33.1, C34.1, H5.2, H5.4, H5.6, H5.8, H8.3, R41.1, U5.OUT, U6.AVCC, U6.DVCC; no longer C20.1, C21.1, C22.1, C28.1, H4.2, H4.4, H4.6, H4.8, H5.3, R19.1, U4.OUT, U5.AVCC, U5.DVCC
- net +5V: now also C22.1, C23.1, C29.1, C30.1, H4.2, H4.4, H4.6, H4.8, R30.1, R33.2, U5.EN, U5.IN; no longer C1.1, C19.1, C2.1, C4.1, H3.2, H3.4, H3.6, H3.8, R1.1, R75.2, U3.IN, U4.EN
- net +VE: now also C15.1, C17.1, U3G$3.V+; no longer C39.1, C41.1, U7G$3.V+
- net -VE: now also C16.2, C18.2, U3G$3.V-; no longer C40.2, C42.2, U7G$3.V-
- net AVCC: now also H1.1, H1.2; no longer H9.1, H9.2
- net CH10_CV: now also R26.1, U1G$1.IN-, U1G$1.OUT; no longer R6.1, U2G$1.IN-, U2G$1.OUT
- net CH11_CV: now also R40.2, U1G$2.IN-, U1G$2.OUT; no longer R12.2, U2G$2.IN-, U2G$2.OUT
- net CH12_CV: now also R39.2, U2G1.IN-, U2G1.OUT; no longer R10.2, U1G1.IN-, U1G1.OUT
- net CH13_CV: now also R38.2, U2G2.IN-, U2G2.OUT; no longer R8.2, U1G2.IN-, U1G2.OUT
- net CH14_CV: now also R24.1, U2G3.IN-, U2G3.OUT; no longer R4.1, U1G3.IN-, U1G3.OUT
- net CH15_CV: now also R25.1, U2G4.IN-, U2G4.OUT; no longer R5.1, U1G4.IN-, U1G4.OUT
- net CH15_CV_IN: now also C8.1, JP1.3, R6.2, U2G4.IN+; no longer C17.1, JP3.3, R18.2, U1G4.IN+
- net CH15_GK_VOL: now also JP1.1, R20.1; no longer JP3.1, R24.1
- net CH15_GK_VOL/CV: now also H3.8, JP1.2; no longer H8.8, JP3.2
- net CH1_GK: now also H2.1, R7.2; no longer H6.1, R30.2
- net CH2_GK: now also H2.2, R8.2; no longer H6.2, R32.2
- net CH3_GK: now also H2.3, R9.2; no longer H6.3, R34.2
- net CH4_GK: now also H2.4, R10.2; no longer H6.4, R36.2
- net CH5_GK: now also H2.5, R11.2; no longer H6.5, R38.2
- net CH6_GK: now also H2.6, R12.2; no longer H6.6, R40.2
- net CH7_CV_IN: now also H6.4, U6.P2.1; no longer H1.4, U5.P2.1
- net CH7_GK_SW/CV: now also H2.8; no longer H6.8
- net CH8_CV_IN: now also H6.5, JP3.3, U6.P2.2; no longer H1.5, JP1.3, U5.P2.2
- net CH8_GK_SW: now also JP3.1; no longer JP1.1
- net CH8_GK_SW/CV: now also H3.1, JP3.2; no longer H8.1, JP1.2
- net CH9_CV: now also H3.2, U6.P2.0; no longer H8.2, U5.P2.0
- net DVCC: now also H1.5, H1.6; no longer H9.5, H9.6
- net D_VIN: now also C2.+, C27.1, C28.1, U4.OUT; no longer C27.+, C44.1, C9.1, U3.OUT
- net GK_VOL: now also R23.2; no longer R25.2
- net GND: now also C1.-, C16.1, C18.1, C2.-, C26.2, C27.2, C29.2, C30.2, C31.2, C32.2, C33.2, C34.2, C35.2, C36.1, C37.1, H1.3, H1.4, H1.7, H1.8, H5.1, H5.3, H5.5, H5.7, H7.7, H7.8, H8.4, R1.1, R2.1, R21.2, R27.2, R29.2, R3.1, R35.2, R36.2, R37.2, R4.1, R5.1, R6.1, U1G$3.V-, U2P1.V-, U4.GND1, U5.GND, U6.AVSS, U6.DVSS; no longer C1.2, C13.2, C16.2, C18.2, C2.2, C26.-, C27.-, C29.1, C30.1, C39.2, C40.1, C41.2, C42.1, C43.2, C44.2, H2.7, H2.8, H3.1, H3.3, H3.5, H3.7, H5.4, H9.3, H9.4, H9.7, H9.8, R11.2, R29.1, R31.1, R33.1, R35.1, R37.1, R39.1, R55.2, R56.2, R57.2, R7.2, R9.2, U1P1.V-, U2G$3.V-, U3.GND, U3.GND1, U5.AVSS, U5.DVSS
- net MONO_GK: now also H2.7, R19.1; no longer H6.7, R26.1
- net N$1: now also R31.2; no longer R2.2
- net N$10: now also C3.1, H3.3, R1.2, U1G$1.IN+; no longer C10.1, H8.3, R13.2, U2G$1.IN+
- net N$11: now also C4.1, H3.4, R2.2, U1G$2.IN+; no longer C11.1, H8.4, R14.2, U2G$2.IN+
- net N$14: now also C5.1, H3.5, R3.2, U2G1.IN+; no longer C14.1, H8.5, R15.2, U1G1.IN+
- net N$19: now also C6.1, H3.6, R4.2, U2G2.IN+; no longer C15.1, H8.6, R16.2, U1G2.IN+
- net N$2: now also R31.1; no longer R2.1
- net N$20: now also C7.1, H3.7, R5.2, U2G3.IN+; no longer C16.1, H8.7, R17.2, U1G3.IN+
- net N$21: now also R22.1; no longer R27.1
- net N$3: now also R32.2; no longer R3.2
- net N$35: now also R23.1, U3G$2.IN-, U3G$2.OUT; no longer R25.1, U7G$2.IN-, U7G$2.OUT
- net N$36: now also C14.1, R20.2, U3G$2.IN+; no longer C43.1, R24.2, U7G$2.IN+
- net N$37: now also C13.2, R19.2; no longer C31.2, R26.2
- net N$38: now also C13.1, R21.1, U3G$1.IN+; no longer C31.1, R28.1, U7G$1.IN+
- net N$39: now also R22.2, U3G$1.IN-, U3G$1.OUT; no longer R27.2, U7G$1.IN-, U7G$1.OUT
- net N$42: now also R13.2, R7.1; no longer R29.2, R30.1
- net N$43: now also R14.2, R8.1; no longer R31.2, R32.1
- net N$44: now also R15.2, R9.1; no longer R33.2, R34.1
- net N$45: now also R10.1, R16.2; no longer R35.2, R36.1
- net N$46: now also R11.1, R17.2; no longer R37.2, R38.1
- net N$47: now also R12.1, R18.2; no longer R39.2, R40.1
- net N$5: now also R30.2; no longer R1.2
- net N$6: now also U6.NC_2; no longer U5.NC_2
- net N$8: now also R34.2; no longer R74.2
- net N$9: now also R32.1, R33.1; no longer R3.1, R75.1
- net NC: now also U6.NC_1; no longer U5.NC_1
- net P1.0: now also C21.1, R26.2, R29.1, U6.P1.0; no longer C25.1, R57.1, R6.2, U5.P1.0
- net P1.1: now also H6.1, U6.P1.1; no longer H1.1, U5.P1.1
- net P1.2: now also R34.1, U6.P1.2; no longer R74.1, U5.P1.2
- net P1.3: now also C26.1, R37.1, R40.1, U6.P1.3; no longer C5.1, R11.1, R12.1, U5.P1.3
- net P1.4: now also C25.1, R36.1, R39.1, U6.P1.4; no longer C13.1, R10.1, R9.1, U5.P1.4
- net P1.5: now also C24.1, R35.1, R38.1, U6.P1.5; no longer C12.1, R7.1, R8.1, U5.P1.5
- net P1.6: now also C19.1, R24.2, R27.1, U6.P1.6; no longer C23.1, R4.2, R55.1, U5.P1.6
- net P1.7: now also C20.1, R25.2, R28.1, U6.P1.7; no longer C24.1, R5.2, R56.1, U5.P1.7
- net P2.3: now also H7.1, U6.P2.3; no longer H2.1, U5.P2.3
- net P2.4: now also H7.2, U6.P2.4; no longer H2.2, U5.P2.4
- net P2.5: now also H7.3, U6.P2.5; no longer H2.3, U5.P2.5
- net P2.6: now also C37.2, U6.P2.6; no longer C29.2, U5.P2.6
- net P2.7: now also C36.2, U6.P2.7; no longer C30.2, U5.P2.7
- net P3.0: now also H6.3, U6.P3.0; no longer H1.3, U5.P3.0
- net P3.1: now also H6.2, U6.P3.1; no longer H1.2, U5.P3.1
- net P3.2: now also H6.6, U6.P3.2; no longer H1.6, U5.P3.2
- net P3.3: now also H6.7, U6.P3.3; no longer H1.7, U5.P3.3
- net P3.4: now also H6.8, U6.P3.4; no longer H1.8, U5.P3.4
- net P3.5: now also H7.4, U6.P3.5; no longer H2.4, U5.P3.5
- net P3.6: now also H7.5, U6.P3.6; no longer H2.5, U5.P3.6
- net P3.7: now also H7.6, U6.P3.7; no longer H2.6, U5.P3.7
- net TEST: now also H8.1, U6.TEST; no longer H5.1, U5.TEST
- net VIN: now also C1.+, C10.1, C11.1, C12.1, C9.1, U1G$3.V+, U2P1.V+; no longer C26.+, C3.1, C6.1, C7.1, C8.1, U1P1.V+, U2G$3.V+

Commit message: update shematic pdf
Parts:
- removed U$1: 13P-MIDI, CYCFI_Con:13P-MIDI
- added 13P-CN1: 13P-MIDI, CYCFI_Con:13P-MIDI
- R10, R11, R12, R13, R14, R15, R16, R17, R18, R7, R8, R9: value 5k -> 5.1k
- renumbered Q1 to X1
Connections:
- net +VE: now also 13P-CN1.12; no longer U$1.12
- net -VE: now also 13P-CN1.13; no longer U$1.13
- net CH7_GK_SW: now also 13P-CN1.10; no longer U$1.10
- net CH8_GK_SW: now also 13P-CN1.11; no longer U$1.11
- net GK_VOL: now also 13P-CN1.8; no longer U$1.8
- net GND: now also 13P-CN1.14, 13P-CN1.15; no longer U$1.14, U$1.15
- net N$21: now also 13P-CN1.7; no longer U$1.7
- net N$42: now also 13P-CN1.1; no longer U$1.1
- net N$43: now also 13P-CN1.2; no longer U$1.2
- net N$44: now also 13P-CN1.3; no longer U$1.3
- net N$45: now also 13P-CN1.4; no longer U$1.4
- net N$46: now also 13P-CN1.5; no longer U$1.5
- net N$47: now also 13P-CN1.6; no longer U$1.6
Other:
- note removed: "MCU INTERFACE:CONTROL VOLTAGES (CH9 - CH15)"
- moved on the sheet: C13, C14, C15, C16, C17, C18, D1, D2, R10, R11, R12, R13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
