File: breakout_box/gk_+_midi_module/gk+midi board v2.5.sch (EAGLE design)
At the start: 114 parts, among them T1 2N2222, T2 2N2222, U2 LMV324, U3 TLV2170DGKT, U4 L78LXX, U5 MIC5205-3.3, U6 MSP430G2553RHB32, X1 QUARZ5

Commit message: updates
Parts:
- renumbered U6 to U6B
Other:
- note added: "AUXILLIARY PINS"
- note added: "MCU Power/ Programming Pins/ Aux Pins"
- note added: "MSP430G2553RHB32"
- note added: "U6A"
- note removed: "Digital Power Source"
- note removed: "MCU MODULE"

Commit message: updates
Connections:
- net CH7_CV_IN renamed CH7_SW
- net CH8_CV_IN renamed CH8_SW
- net CH9_CV renamed CH9_SW
Changed lines of the file:
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@@
 </busses>
 <nets>
-<net name="CH9_CV" class="0">
+<net name="CH9_SW" class="0">
 <segment>
 <wire x1="116.205" y1="139.065" x2="136.525" y2="139.065" width="0.1524" layer="91"/>
@@
 </segment>
 </net>
-<net name="CH8_CV_IN" class="0">
+<net name="CH8_SW" class="0">
 <segment>
 <pinref part="JP3" gate="A" pin="3"/>
@@
 </segment>
 </net>
-<net name="CH7_CV_IN" class="0">
+<net name="CH7_SW" class="0">
 <segment>
 <pinref part="JP2" gate="A" pin="3"/>
@@
 </busses>
 <nets>
-<net name="CH9_CV" class="0">
+<net name="CH9_SW" class="0">
 <segment>
 <label x="189.865" y="166.6875" size="1.778" layer="95"/>
@@
 </segment>
 </net>
-<net name="CH8_CV_IN" class="0">
+<net name="CH8_SW" class="0">
 <segment>
 <wire x1="152.4" y1="118.11" x2="165.735" y2="118.11" width="0.1524" layer="91"/>
@@
 </segment>
 </net>
-<net name="CH7_CV_IN" class="0">
+<net name="CH7_SW" class="0">
 <segment>
 <wire x1="152.4" y1="115.57" x2="168.275" y2="115.57" width="0.1524" layer="91"/>
@@
 </segment>
 </net>
-<net name="CH7_CV_IN" class="0">
+<net name="CH7_SW" class="0">
 <segment>
 <pinref part="U6B" gate="G$1" pin="P2.1"/>
@@
 </segment>
 </net>
-<net name="CH9_CV" class="0">
+<net name="CH9_SW" class="0">
 <segment>
 <pinref part="U6B" gate="G$1" pin="P2.0"/>
@@
 </segment>
 </net>
-<net name="CH8_CV_IN" class="0">
+<net name="CH8_SW" class="0">
 <segment>
 <pinref part="U6B" gate="G$1" pin="P2.2"/>
