File: breakout_box/gk_+_midi_module/gk+midi board v2.5.brd (EAGLE design)
At the start: 65.2 x 100 mm, 114 parts, among them T1 2N2222, T2 2N2222, U2 LMV324, U3 TLV2170DGKT, U4 L78LXX, U5 MIC5205-3.3, U6 MSP430G2553RHB32, X1 QUARZ5

Commit message: updates
Changed lines of the file:
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@@
 <text x="54.5" y="19.75" size="0.7" layer="25" font="vector" ratio="12">GND</text>
 <text x="59.75" y="19.75" size="0.7" layer="25" font="vector" ratio="12">GND</text>
-<text x="40.75" y="72.25" size="0.7" layer="25" font="vector" ratio="12" rot="R90">TEST</text>
-<text x="43.25" y="72" size="0.7" layer="25" font="vector" ratio="12" rot="R90">/RST</text>
-<text x="45.75" y="72.25" size="0.7" layer="25" font="vector" ratio="12" rot="R90">DVCC</text>
-<text x="48.25" y="72.25" size="0.7" layer="25" font="vector" ratio="12" rot="R90">DGND</text>
+<text x="40.625" y="72.5" size="0.7" layer="25" font="vector" ratio="12" rot="R90">TEST</text>
+<text x="43.25" y="72.375" size="0.7" layer="25" font="vector" ratio="12" rot="R90">/RST</text>
+<text x="45.75" y="72.625" size="0.7" layer="25" font="vector" ratio="12" rot="R90">DVCC</text>
+<text x="48.25" y="72.5" size="0.7" layer="25" font="vector" ratio="12" rot="R90">DGND</text>
 <text x="48" y="27.25" size="0.7" layer="25" font="vector" ratio="12">P1.1</text>
 <text x="48" y="29.75" size="0.7" layer="25" font="vector" ratio="12">P3.1</text>

Commit message: updates
Parts:
- renumbered U6 to U6B
Changed lines of the file:
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@@
 <attribute name="VALUE" x="35.405" y="62.115" size="0.8062" layer="27" rot="R90"/>
 </element>
-<element name="U6" library="CYCFI_IC" package="QFN32" value="MSP430G2553RHB32" x="42" y="58.5" smashed="yes" rot="R90">
+<element name="U6B" library="CYCFI_IC" package="QFN32" value="MSP430G2553RHB32" x="42" y="58.5" smashed="yes" rot="R90">
 <attribute name="VALUE" x="46.35" y="54.45" size="0.8062" layer="27" rot="R90"/>
 <attribute name="NAME" x="38.55" y="56.75" size="0.8062" layer="25" font="vector" rot="R180"/>
@@
 <wire x1="14.75" y1="49.25" x2="15.93" y2="49.25" width="0.2032" layer="1"/>
 <wire x1="15.93" y1="49.25" x2="16.35" y2="49.67" width="0.2032" layer="1"/>
-<contactref element="U6" pad="9"/>
+<contactref element="U6B" pad="9"/>
 <wire x1="44.4905" y1="56.75" x2="45" y2="56.75" width="0.2032" layer="1"/>
 <wire x1="45" y1="56.75" x2="45.25" y2="56.5" width="0.2032" layer="1"/>
@@
 <contactref element="C34" pad="2"/>
 <contactref element="C30" pad="2"/>
-<contactref element="U6" pad="28"/>
-<contactref element="U6" pad="27"/>
+<contactref element="U6B" pad="28"/>
+<contactref element="U6B" pad="27"/>
 <contactref element="C35" pad="2"/>
 <contactref element="C37" pad="1"/>
@@
 <signal name="CH8_CV_IN">
 <contactref element="JP3" pad="3"/>
-<contactref element="U6" pad="11"/>
+<contactref element="U6B" pad="11"/>
 <contactref element="H6" pad="5"/>
 <wire x1="44.4905" y1="57.75" x2="46.5" y2="57.75" width="0.2032" layer="1"/>
@@
 <signal name="CH7_CV_IN">
 <contactref element="JP2" pad="3"/>
-<contactref element="U6" pad="10"/>
+<contactref element="U6B" pad="10"/>
 <contactref element="H6" pad="4"/>
 <wire x1="44.4905" y1="57.25" x2="45.75" y2="57.25" width="0.2032" layer="1"/>
@@
 </signal>
 <signal name="!RST">
-<contactref element="U6" pad="23"/>
+<contactref element="U6B" pad="23"/>
 <contactref element="R41" pad="2"/>
 <contactref element="C35" pad="1"/>
@@
 </signal>
 <signal name="TEST">
-<contactref element="U6" pad="24"/>
+<contactref element="U6B" pad="24"/>
 <contactref element="H8" pad="1"/>
 <via x="40.25" y="65.75" extent="1-16" drill="0.4"/>
@@
 </signal>
 <signal name="+3.3V">
-<contactref element="U6" pad="30"/>
+<contactref element="U6B" pad="30"/>
 <contactref element="R41" pad="1"/>
-<contactref element="U6" pad="29"/>
+<contactref element="U6B" pad="29"/>
 <contactref element="C33" pad="1"/>
 <contactref element="C34" pad="1"/>
@@
 <signal name="P1.1">
 <contactref element="H6" pad="1"/>
-<contactref element="U6" pad="1"/>
+<contactref element="U6B" pad="1"/>
 <wire x1="40.25" y1="56.0095" x2="40.25" y2="56" width="0.2032" layer="1"/>
 <wire x1="40.25" y1="56" x2="39.75" y2="55.5" width="0.2032" layer="1"/>
@@
 </signal>
 <signal name="P3.2">
-<contactref element="U6" pad="12"/>
+<contactref element="U6B" pad="12"/>
 <contactref element="H6" pad="6"/>
 <wire x1="52" y1="40.31" x2="50.44" y2="40.31" width="0.2032" layer="1"/>
@@
 </signal>
 <signal name="P3.3">
-<contactref element="U6" pad="13"/>
+<contactref element="U6B" pad="13"/>
 <contactref element="H6" pad="7"/>
 <wire x1="44.4905" y1="58.75" x2="51.25" y2="58.75" width="0.2032" layer="1"/>
@@
 </signal>
 <signal name="P3.4">
-<contactref element="U6" pad="14"/>
+<contactref element="U6B" pad="14"/>
 <contactref element="H6" pad="8"/>
 <wire x1="44.4905" y1="59.25" x2="51.5" y2="59.25" width="0.2032" layer="1"/>
@@
 </signal>
 <signal name="P2.3">
-<contactref element="U6" pad="15"/>
+<contactref element="U6B" pad="15"/>
 <contactref element="H7" pad="1"/>
 <wire x1="54.875" y1="58.375" x2="53.5" y2="59.75" width="0.2032" layer="1"/>
@@
 </signal>
 <signal name="P2.4">
-<contactref element="U6" pad="16"/>
+<contactref element="U6B" pad="16"/>
 <contactref element="H7" pad="2"/>
 <wire x1="44.4905" y1="60.25" x2="54.25" y2="60.25" width="0.2032" layer="1"/>
@@
 </signal>
 <signal name="P2.5">
-<contactref element="U6" pad="17"/>
+<contactref element="U6B" pad="17"/>
 <contactref element="H7" pad="3"/>
 <wire x1="55.75" y1="40.31" x2="56.81" y2="40.31" width="0.2032" layer="1"/>
@@
 </signal>
 <signal name="P3.5">
-<contactref element="U6" pad="18"/>
+<contactref element="U6B" pad="18"/>
 <contactref element="H7" pad="4"/>
 <wire x1="55.75" y1="37.77" x2="56.27" y2="37.77" width="0.2032" layer="1"/>
@@
 </signal>
 <signal name="P3.6">
-<contactref element="U6" pad="19"/>
+<contactref element="U6B" pad="19"/>
 <contactref element="H7" pad="5"/>
 <wire x1="55.75" y1="35.23" x2="56.23" y2="35.23" width="0.2032" layer="1"/>
@@
 </signal>
 <signal name="P3.7">
-<contactref element="U6" pad="20"/>
+<contactref element="U6B" pad="20"/>
 <contactref element="H7" pad="6"/>
 <wire x1="42.25" y1="60.9905" x2="42.25" y2="62.25" width="0.2032" layer="1"/>
@@
 </signal>
 <signal name="P1.2">
-<contactref element="U6" pad="2"/>
+<contactref element="U6B" pad="2"/>
 <contactref element="R34" pad="1"/>
 <contactref element="TP_SER" pad="TP"/>
@@
 </signal>
 <signal name="P1.3">
-<contactref element="U6" pad="3"/>
+<contactref element="U6B" pad="3"/>
 <contactref element="R37" pad="1"/>
 <contactref element="C26" pad="1"/>
@@
 </signal>
 <signal name="P1.4">
-<contactref element="U6" pad="4"/>
+<contactref element="U6B" pad="4"/>
 <contactref element="R36" pad="1"/>
 <contactref element="C25" pad="1"/>
@@
 </signal>
 <signal name="P1.5">
-<contactref element="U6" pad="5"/>
+<contactref element="U6B" pad="5"/>
 <contactref element="R35" pad="1"/>
 <contactref element="C24" pad="1"/>
@@
 </signal>
 <signal name="P3.1">
-<contactref element="U6" pad="6"/>
+<contactref element="U6B" pad="6"/>
 <contactref element="H6" pad="2"/>
 <wire x1="42.75" y1="56.0095" x2="42.75" y2="54.25" width="0.2032" layer="1"/>
@@
 </signal>
 <signal name="P3.0">
-<contactref element="U6" pad="7"/>
+<contactref element="U6B" pad="7"/>
 <contactref element="H6" pad="3"/>
 <wire x1="52" y1="32.69" x2="49.56" y2="32.69" width="0.2032" layer="1"/>
@@
 </signal>
 <signal name="NC">
-<contactref element="U6" pad="8"/>
+<contactref element="U6B" pad="8"/>
 </signal>
 <signal name="P1.6">
-<contactref element="U6" pad="21"/>
+<contactref element="U6B" pad="21"/>
 <contactref element="R27" pad="1"/>
 <contactref element="C19" pad="1"/>
@@
 </signal>
 <signal name="P1.7">
-<contactref element="U6" pad="22"/>
+<contactref element="U6B" pad="22"/>
 <contactref element="R28" pad="1"/>
 <contactref element="C20" pad="1"/>
@@
 </signal>
 <signal name="P2.7">
-<contactref element="U6" pad="25"/>
+<contactref element="U6B" pad="25"/>
 <contactref element="X1" pad="2"/>
 <contactref element="C36" pad="2"/>
@@
 </signal>
 <signal name="P2.6">
-<contactref element="U6" pad="26"/>
+<contactref element="U6B" pad="26"/>
 <contactref element="C37" pad="2"/>
 <contactref element="X1" pad="1"/>
@@
 </signal>
 <signal name="P1.0">
-<contactref element="U6" pad="31"/>
+<contactref element="U6B" pad="31"/>
 <contactref element="R29" pad="1"/>
 <contactref element="C21" pad="1"/>
@@
 </signal>
 <signal name="N$6">
-<contactref element="U6" pad="32"/>
+<contactref element="U6B" pad="32"/>
 </signal>
 <signal name="N$3">

Commit message: updates
Connections:
- net CH7_CV_IN renamed CH7_SW
- net CH8_CV_IN renamed CH8_SW
- net CH9_CV renamed CH9_SW
Changed lines of the file:
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@@
 </elements>
 <signals>
-<signal name="CH9_CV">
+<signal name="CH9_SW">
 <contactref element="TP_1" pad="TP"/>
 <contactref element="H3" pad="2"/>
@@
 <via x="2" y="87.375" extent="1-16" drill="0.4"/>
 </signal>
-<signal name="CH8_CV_IN">
+<signal name="CH8_SW">
 <contactref element="JP3" pad="3"/>
 <contactref element="U6B" pad="11"/>
@@
 <wire x1="49.75" y1="57" x2="47.25" y2="57" width="0.2032" layer="1"/>
 </signal>
-<signal name="CH7_CV_IN">
+<signal name="CH7_SW">
 <contactref element="JP2" pad="3"/>
 <contactref element="U6B" pad="10"/>
