File: breakout_box/gk_+_midi_module/gk+midi_module.brd (EAGLE design)
At the start: 65.2 x 100 mm, 114 parts, among them T1 2N2222, T2 2N2222, U2 LMV324, U3 TLV2170DGKT, U4 L78LXX, U5 MIC5205-3.3, U6B MSP430G2553RHB32, X1 QUARZ5

Commit message: update schematics
Parts:
- renumbered U6B to U6
Other:
- board text added: "P2.1/ AUX1"
- board text added: "P2.2/ AUX2"
- board text added: "P2.3/ AUX3"
- board text added: "P2.4/ AUX4"
- board text added: "P2.5/ AUX5"
- board text added: "P3.6/ AUX6"
- board text removed: "P2.1"
- board text removed: "P2.2"
- board text removed: "P2.3"
- board text removed: "P2.4"
- board text removed: "P2.5"
- board text removed: "P3.6"
Changed lines of the file:
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@@
 <layer number="220" name="220bmp" color="21" fill="1" visible="no" active="no"/>
 <layer number="221" name="221bmp" color="22" fill="1" visible="no" active="no"/>
-<layer number="222" name="222bmp" color="23" fill="1" visible="no" active="no"/>
 <layer number="223" name="223bmp" color="24" fill="1" visible="no" active="no"/>
 <layer number="224" name="224bmp" color="25" fill="1" visible="no" active="no"/>
@@
 <text x="48" y="29.75" size="0.7" layer="25" font="vector" ratio="12">P3.1</text>
 <text x="48" y="32.25" size="0.7" layer="25" font="vector" ratio="12">P3.0</text>
-<text x="48" y="35" size="0.7" layer="25" font="vector" ratio="12">P2.1</text>
-<text x="48" y="37.5" size="0.7" layer="25" font="vector" ratio="12">P2.2</text>
+<text x="47.375" y="34.375" size="0.7" layer="25" font="vector" ratio="12">P2.1/
+AUX1</text>
+<text x="47.375" y="36.875" size="0.7" layer="25" font="vector" ratio="12">P2.2/
+AUX2</text>
 <text x="48" y="40" size="0.7" layer="25" font="vector" ratio="12">P3.2</text>
 <text x="48" y="42.5" size="0.7" layer="25" font="vector" ratio="12">P3.3</text>
 <text x="48" y="45" size="0.7" layer="25" font="vector" ratio="12">P3.4</text>
-<text x="58" y="45" size="0.7" layer="25" font="vector" ratio="12">P2.3</text>
-<text x="58" y="42.5" size="0.7" layer="25" font="vector" ratio="12">P2.4</text>
-<text x="58" y="40" size="0.7" layer="25" font="vector" ratio="12">P2.5</text>
+<text x="58" y="44.625" size="0.7" layer="25" font="vector" ratio="12">P2.3/
+AUX3</text>
+<text x="58" y="41.875" size="0.7" layer="25" font="vector" ratio="12">P2.4/
+AUX4</text>
+<text x="58" y="39.375" size="0.7" layer="25" font="vector" ratio="12">P2.5/
+AUX5</text>
 <text x="58" y="37.5" size="0.7" layer="25" font="vector" ratio="12">P3.5</text>
-<text x="58" y="35" size="0.7" layer="25" font="vector" ratio="12">P3.6</text>
+<text x="58" y="34.5" size="0.7" layer="25" font="vector" ratio="12">P3.6/
+AUX6</text>
 <text x="58" y="32.25" size="0.7" layer="25" font="vector" ratio="12">P3.7</text>
 <text x="58" y="29.75" size="0.7" layer="25" font="vector" ratio="12">GND</text>
@@
 <attribute name="VALUE" x="35.405" y="62.115" size="0.8062" layer="27" rot="R90"/>
 </element>
-<element name="U6B" library="CYCFI_IC" package="QFN32" value="MSP430G2553RHB32" x="42" y="58.5" smashed="yes" rot="R90">
+<element name="U6" library="CYCFI_IC" package="QFN32" value="MSP430G2553RHB32" x="42" y="58.5" smashed="yes" rot="R90">
 <attribute name="VALUE" x="46.35" y="54.45" size="0.8062" layer="27" rot="R90"/>
 <attribute name="NAME" x="38.55" y="56.75" size="0.8062" layer="25" font="vector" rot="R180"/>
@@
 <wire x1="14.75" y1="49.25" x2="15.93" y2="49.25" width="0.2032" layer="1"/>
 <wire x1="15.93" y1="49.25" x2="16.35" y2="49.67" width="0.2032" layer="1"/>
-<contactref element="U6B" pad="9"/>
+<contactref element="U6" pad="9"/>
 <wire x1="44.4905" y1="56.75" x2="45" y2="56.75" width="0.2032" layer="1"/>
 <wire x1="45" y1="56.75" x2="45.25" y2="56.5" width="0.2032" layer="1"/>
@@
 <contactref element="C34" pad="2"/>
 <contactref element="C30" pad="2"/>
-<contactref element="U6B" pad="28"/>
-<contactref element="U6B" pad="27"/>
+<contactref element="U6" pad="28"/>
+<contactref element="U6" pad="27"/>
 <contactref element="C35" pad="2"/>
 <contactref element="C37" pad="1"/>
@@
 <signal name="CH8_SW">
 <contactref element="JP3" pad="3"/>
-<contactref element="U6B" pad="11"/>
+<contactref element="U6" pad="11"/>
 <contactref element="H6" pad="5"/>
 <wire x1="44.4905" y1="57.75" x2="46.5" y2="57.75" width="0.2032" layer="1"/>
@@
 <signal name="CH7_SW">
 <contactref element="JP2" pad="3"/>
-<contactref element="U6B" pad="10"/>
+<contactref element="U6" pad="10"/>
 <contactref element="H6" pad="4"/>
 <wire x1="44.4905" y1="57.25" x2="45.75" y2="57.25" width="0.2032" layer="1"/>
@@
 </signal>
 <signal name="!RST">
-<contactref element="U6B" pad="23"/>
+<contactref element="U6" pad="23"/>
 <contactref element="R41" pad="2"/>
 <contactref element="C35" pad="1"/>
@@
 </signal>
 <signal name="TEST">
-<contactref element="U6B" pad="24"/>
+<contactref element="U6" pad="24"/>
 <contactref element="H8" pad="1"/>
 <via x="40.25" y="65.75" extent="1-16" drill="0.4"/>
@@
 </signal>
 <signal name="+3.3V">
-<contactref element="U6B" pad="30"/>
+<contactref element="U6" pad="30"/>
 <contactref element="R41" pad="1"/>
-<contactref element="U6B" pad="29"/>
+<contactref element="U6" pad="29"/>
 <contactref element="C33" pad="1"/>
 <contactref element="C34" pad="1"/>
@@
 <signal name="P1.1">
 <contactref element="H6" pad="1"/>
-<contactref element="U6B" pad="1"/>
+<contactref element="U6" pad="1"/>
 <wire x1="40.25" y1="56.0095" x2="40.25" y2="56" width="0.2032" layer="1"/>
 <wire x1="40.25" y1="56" x2="39.75" y2="55.5" width="0.2032" layer="1"/>
@@
 </signal>
 <signal name="P3.2">
-<contactref element="U6B" pad="12"/>
+<contactref element="U6" pad="12"/>
 <contactref element="H6" pad="6"/>
 <wire x1="52" y1="40.31" x2="50.44" y2="40.31" width="0.2032" layer="1"/>
@@
 </signal>
 <signal name="P3.3">
-<contactref element="U6B" pad="13"/>
+<contactref element="U6" pad="13"/>
 <contactref element="H6" pad="7"/>
 <wire x1="44.4905" y1="58.75" x2="51.25" y2="58.75" width="0.2032" layer="1"/>
@@
 </signal>
 <signal name="P3.4">
-<contactref element="U6B" pad="14"/>
+<contactref element="U6" pad="14"/>
 <contactref element="H6" pad="8"/>
 <wire x1="44.4905" y1="59.25" x2="51.5" y2="59.25" width="0.2032" layer="1"/>
@@
 </signal>
 <signal name="P2.3">
-<contactref element="U6B" pad="15"/>
+<contactref element="U6" pad="15"/>
 <contactref element="H7" pad="1"/>
 <wire x1="54.875" y1="58.375" x2="53.5" y2="59.75" width="0.2032" layer="1"/>
@@
 </signal>
 <signal name="P2.4">
-<contactref element="U6B" pad="16"/>
+<contactref element="U6" pad="16"/>
 <contactref element="H7" pad="2"/>
 <wire x1="44.4905" y1="60.25" x2="54.25" y2="60.25" width="0.2032" layer="1"/>
@@
 </signal>
 <signal name="P2.5">
-<contactref element="U6B" pad="17"/>
+<contactref element="U6" pad="17"/>
 <contactref element="H7" pad="3"/>
 <wire x1="55.75" y1="40.31" x2="56.81" y2="40.31" width="0.2032" layer="1"/>
@@
 </signal>
 <signal name="P3.5">
-<contactref element="U6B" pad="18"/>
+<contactref element="U6" pad="18"/>
 <contactref element="H7" pad="4"/>
 <wire x1="55.75" y1="37.77" x2="56.27" y2="37.77" width="0.2032" layer="1"/>
@@
 </signal>
 <signal name="P3.6">
-<contactref element="U6B" pad="19"/>
+<contactref element="U6" pad="19"/>
 <contactref element="H7" pad="5"/>
 <wire x1="55.75" y1="35.23" x2="56.23" y2="35.23" width="0.2032" layer="1"/>
@@
 </signal>
 <signal name="P3.7">
-<contactref element="U6B" pad="20"/>
+<contactref element="U6" pad="20"/>
 <contactref element="H7" pad="6"/>
 <wire x1="42.25" y1="60.9905" x2="42.25" y2="62.25" width="0.2032" layer="1"/>
@@
 </signal>
 <signal name="P1.2">
-<contactref element="U6B" pad="2"/>
+<contactref element="U6" pad="2"/>
 <contactref element="R34" pad="1"/>
 <contactref element="TP_SER" pad="TP"/>
@@
 </signal>
 <signal name="P1.3">
-<contactref element="U6B" pad="3"/>
+<contactref element="U6" pad="3"/>
 <contactref element="R37" pad="1"/>
 <contactref element="C26" pad="1"/>
@@
 </signal>
 <signal name="P1.4">
-<contactref element="U6B" pad="4"/>
+<contactref element="U6" pad="4"/>
 <contactref element="R36" pad="1"/>
 <contactref element="C25" pad="1"/>
@@
 </signal>
 <signal name="P1.5">
-<contactref element="U6B" pad="5"/>
+<contactref element="U6" pad="5"/>
 <contactref element="R35" pad="1"/>
 <contactref element="C24" pad="1"/>
@@
 </signal>
 <signal name="P3.1">
-<contactref element="U6B" pad="6"/>
+<contactref element="U6" pad="6"/>
 <contactref element="H6" pad="2"/>
 <wire x1="42.75" y1="56.0095" x2="42.75" y2="54.25" width="0.2032" layer="1"/>
@@
 </signal>
 <signal name="P3.0">
-<contactref element="U6B" pad="7"/>
+<contactref element="U6" pad="7"/>
 <contactref element="H6" pad="3"/>
 <wire x1="52" y1="32.69" x2="49.56" y2="32.69" width="0.2032" layer="1"/>
@@
 </signal>
 <signal name="NC">
-<contactref element="U6B" pad="8"/>
+<contactref element="U6" pad="8"/>
 </signal>
 <signal name="P1.6">
-<contactref element="U6B" pad="21"/>
+<contactref element="U6" pad="21"/>
 <contactref element="R27" pad="1"/>
 <contactref element="C19" pad="1"/>
@@
 </signal>
 <signal name="P1.7">
-<contactref element="U6B" pad="22"/>
+<contactref element="U6" pad="22"/>
 <contactref element="R28" pad="1"/>
 <contactref element="C20" pad="1"/>
@@
 </signal>
 <signal name="P2.7">
-<contactref element="U6B" pad="25"/>
+<contactref element="U6" pad="25"/>
 <contactref element="X1" pad="2"/>
 <contactref element="C36" pad="2"/>
@@
 </signal>
 <signal name="P2.6">
-<contactref element="U6B" pad="26"/>
+<contactref element="U6" pad="26"/>
 <contactref element="C37" pad="2"/>
 <contactref element="X1" pad="1"/>
@@
 </signal>
 <signal name="P1.0">
-<contactref element="U6B" pad="31"/>
+<contactref element="U6" pad="31"/>
 <contactref element="R29" pad="1"/>
 <contactref element="C21" pad="1"/>
@@
 </signal>
 <signal name="N$6">
-<contactref element="U6B" pad="32"/>
+<contactref element="U6" pad="32"/>
 </signal>
 <signal name="N$3">

Commit message: update gk+midi files
Parts:
- removed JP1: (no value), pinhead-2:1X03M
Connections:
- net CH7_SW renamed CH7_MIDI_SW
- net CH8_SW renamed CH8_MIDI_SW
- removed net N$10: C3.1, JP1.3, R1.2, U1.3
- removed net N$4: H3.3, JP1.2
- net CH10_GK_VOL: now also C3.1, H3.3, R1.2, U1.3; no longer JP1.1
Routing:
- net CH10_GK_VOL: track 66.8 -> 119.3 mm, vias 1 -> 2
- net N$10: track 36.1 -> 0.00 mm, vias 1 -> 0
- net N$4: track 21.4 -> 0.00 mm
Other:
- board text added: "P2.5"
- board text added: "P3.6"
- board text removed: "P2.5/ AUX5"
- board text removed: "P3.6/ AUX6"
Changed lines of the file:
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@@
 <text x="58" y="41.875" size="0.7" layer="25" font="vector" ratio="12">P2.4/
 AUX4</text>
-<text x="58" y="39.375" size="0.7" layer="25" font="vector" ratio="12">P2.5/
-AUX5</text>
+<text x="57.875" y="39.875" size="0.7" layer="25" font="vector" ratio="12">P2.5</text>
 <text x="58" y="37.5" size="0.7" layer="25" font="vector" ratio="12">P3.5</text>
-<text x="58" y="34.5" size="0.7" layer="25" font="vector" ratio="12">P3.6/
-AUX6</text>
+<text x="57.875" y="34.875" size="0.7" layer="25" font="vector" ratio="12">P3.6</text>
 <text x="58" y="32.25" size="0.7" layer="25" font="vector" ratio="12">P3.7</text>
 <text x="58" y="29.75" size="0.7" layer="25" font="vector" ratio="12">GND</text>
@@
 <attribute name="VALUE" x="19.5" y="55" size="0.8128" layer="27" ratio="10" rot="R90"/>
 </element>
-<element name="JP1" library="pinhead-2" package="1X03M" value="" x="14.25" y="28.25" smashed="yes">
-<attribute name="VALUE" x="19.25" y="27.25" size="0.8128" layer="27" ratio="10" rot="R90"/>
-</element>
 <element name="D1" library="CYCFI_semicon" package="SC70-3" value="1SS302" x="20.25" y="76.5" smashed="yes">
 <attribute name="NAME" x="18.3" y="77.35" size="0.8062" layer="25" font="vector"/>
@@
 <wire x1="29.25" y1="45.25" x2="23" y2="45.25" width="0.2032" layer="1"/>
 </signal>
-<signal name="N$10">
-<contactref element="R1" pad="2"/>
-<contactref element="C3" pad="1"/>
-<contactref element="U1" pad="3"/>
-<wire x1="11.21" y1="44.81" x2="11.25" y2="44.85" width="0.2032" layer="1"/>
-<wire x1="11.25" y1="44.85" x2="12.15" y2="44.85" width="0.2032" layer="1"/>
-<wire x1="12.15" y1="44.85" x2="12.5" y2="44.5" width="0.2032" layer="1"/>
-<wire x1="12.5" y1="44.5" x2="13.35" y2="44.5" width="0.2032" layer="1"/>
-<wire x1="13.35" y1="44.5" x2="13.5" y2="44.65" width="0.2032" layer="1"/>
-<wire x1="21.3" y1="46.575" x2="22.325" y2="46.575" width="0.2032" layer="1"/>
-<wire x1="22.325" y1="46.575" x2="22.5" y2="46.75" width="0.2032" layer="1"/>
-<wire x1="22.5" y1="46.75" x2="22.5" y2="47.75" width="0.2032" layer="1"/>
-<wire x1="22.5" y1="47.75" x2="22.25" y2="48" width="0.2032" layer="1"/>
-<wire x1="22.25" y1="48" x2="15.75" y2="48" width="0.2032" layer="1"/>
-<wire x1="15.75" y1="48" x2="15.25" y2="47.5" width="0.2032" layer="1"/>
-<wire x1="15.25" y1="47.5" x2="15.25" y2="44.75" width="0.2032" layer="1"/>
-<wire x1="15.25" y1="44.75" x2="15" y2="44.5" width="0.2032" layer="1"/>
-<wire x1="15" y1="44.5" x2="13.65" y2="44.5" width="0.2032" layer="1"/>
-<wire x1="13.65" y1="44.5" x2="13.5" y2="44.65" width="0.2032" layer="1"/>
-<contactref element="JP1" pad="3"/>
-<wire x1="16.25" y1="28.25" x2="16.25" y2="33.25" width="0.2032" layer="16"/>
-<wire x1="16.25" y1="33.25" x2="10.75" y2="38.75" width="0.2032" layer="16"/>
-<wire x1="10.75" y1="38.75" x2="10.75" y2="43.75" width="0.2032" layer="16"/>
-<wire x1="10.75" y1="43.75" x2="11.25" y2="44.25" width="0.2032" layer="16"/>
-<via x="11.25" y="44.25" extent="1-16" drill="0.4"/>
-<wire x1="11.25" y1="44.25" x2="11.25" y2="44.85" width="0.2032" layer="1"/>
-</signal>
 <signal name="N$11">
 <contactref element="R2" pad="2"/>
@@
 <via x="2" y="87.375" extent="1-16" drill="0.4"/>
 </signal>
-<signal name="CH8_SW">
+<signal name="CH8_MIDI_SW">
 <contactref element="JP3" pad="3"/>
 <contactref element="U6" pad="11"/>
@@
 <wire x1="49.75" y1="57" x2="47.25" y2="57" width="0.2032" layer="1"/>
 </signal>
-<signal name="CH7_SW">
+<signal name="CH7_MIDI_SW">
 <contactref element="JP2" pad="3"/>
 <contactref element="U6" pad="10"/>
@@
 <wire x1="22.02" y1="11.5" x2="21.5" y2="11.5" width="0.6096" layer="1"/>
 </signal>
-<signal name="N$4">
-<contactref element="H3" pad="3"/>
-<contactref element="JP1" pad="2"/>
-<wire x1="6" y1="44.81" x2="8.44" y2="44.81" width="0.2032" layer="16"/>
-<wire x1="8.44" y1="44.81" x2="9.5" y2="43.75" width="0.2032" layer="16"/>
-<wire x1="9.5" y1="43.75" x2="9.5" y2="37.5" width="0.2032" layer="16"/>
-<wire x1="9.5" y1="37.5" x2="14.25" y2="32.75" width="0.2032" layer="16"/>
-<wire x1="14.25" y1="32.75" x2="14.25" y2="28.25" width="0.2032" layer="16"/>
-</signal>
 <signal name="CH10_GK_VOL">
-<contactref element="JP1" pad="1"/>
 <contactref element="R20" pad="1"/>
-<wire x1="12.25" y1="28.25" x2="3.75" y2="28.25" width="0.2032" layer="16"/>
-<wire x1="3.75" y1="28.25" x2="1.5" y2="30.5" width="0.2032" layer="16"/>
+<wire x1="3.625" y1="28.875" x2="1.5" y2="30.5" width="0.2032" layer="16"/>
 <wire x1="1.5" y1="30.5" x2="1.5" y2="51" width="0.2032" layer="16"/>
 <wire x1="1.5" y1="51" x2="2.25" y2="51.75" width="0.2032" layer="16"/>
@@
 <wire x1="27" y1="61" x2="27" y2="62.65" width="0.2032" layer="1"/>
 <wire x1="27" y1="62.65" x2="26.9" y2="62.75" width="0.2032" layer="1"/>
+<contactref element="H3" pad="3"/>
+<wire x1="6" y1="44.81" x2="8.44" y2="44.81" width="0.2032" layer="16"/>
+<wire x1="8.44" y1="44.81" x2="9.5" y2="43.75" width="0.2032" layer="16"/>
+<contactref element="R1" pad="2"/>
+<contactref element="C3" pad="1"/>
+<contactref element="U1" pad="3"/>
+<wire x1="11.21" y1="44.81" x2="11.25" y2="44.85" width="0.2032" layer="1"/>
+<wire x1="11.25" y1="44.85" x2="12.15" y2="44.85" width="0.2032" layer="1"/>
+<wire x1="12.15" y1="44.85" x2="12.5" y2="44.5" width="0.2032" layer="1"/>
+<wire x1="12.5" y1="44.5" x2="13.35" y2="44.5" width="0.2032" layer="1"/>
+<wire x1="13.35" y1="44.5" x2="13.5" y2="44.65" width="0.2032" layer="1"/>
+<wire x1="21.3" y1="46.575" x2="22.325" y2="46.575" width="0.2032" layer="1"/>
+<wire x1="22.325" y1="46.575" x2="22.5" y2="46.75" width="0.2032" layer="1"/>
+<wire x1="22.5" y1="46.75" x2="22.5" y2="47.75" width="0.2032" layer="1"/>
+<wire x1="22.5" y1="47.75" x2="22.25" y2="48" width="0.2032" layer="1"/>
+<wire x1="22.25" y1="48" x2="15.75" y2="48" width="0.2032" layer="1"/>
+<wire x1="15.75" y1="48" x2="15.25" y2="47.5" width="0.2032" layer="1"/>
+<wire x1="15.25" y1="47.5" x2="15.25" y2="44.75" width="0.2032" layer="1"/>
+<wire x1="15.25" y1="44.75" x2="15" y2="44.5" width="0.2032" layer="1"/>
+<wire x1="15" y1="44.5" x2="13.65" y2="44.5" width="0.2032" layer="1"/>
+<wire x1="13.65" y1="44.5" x2="13.5" y2="44.65" width="0.2032" layer="1"/>
+<wire x1="10.75" y1="43.75" x2="11.25" y2="44.25" width="0.2032" layer="16"/>
+<via x="11.25" y="44.25" extent="1-16" drill="0.4"/>
+<wire x1="11.25" y1="44.25" x2="11.25" y2="44.85" width="0.2032" layer="1"/>
+<wire x1="9.5" y1="43.75" x2="9.5" y2="37.5" width="0.2032" layer="16"/>
+<wire x1="9.5" y1="37.5" x2="16.375" y2="30.625" width="0.2032" layer="16"/>
+<wire x1="16.375" y1="30.625" x2="16.375" y2="24.875" width="0.2032" layer="16"/>
+<wire x1="16.375" y1="24.875" x2="15.75" y2="24.25" width="0.2032" layer="16"/>
+<wire x1="15.75" y1="24.25" x2="12.625" y2="24.25" width="0.2032" layer="16"/>
+<wire x1="12.625" y1="24.25" x2="11.875" y2="25" width="0.2032" layer="16"/>
+<wire x1="11.875" y1="25" x2="11.875" y2="27.375" width="0.2032" layer="16"/>
+<wire x1="11.875" y1="27.375" x2="10" y2="28.875" width="0.2032" layer="16"/>
+<wire x1="10" y1="28.875" x2="3.625" y2="28.875" width="0.2032" layer="16"/>
+<wire x1="10.75" y1="43.75" x2="9.5" y2="43.75" width="0.2032" layer="16"/>
 </signal>
 </signals>
