File: breakout_box/io_module/io_module.sch (EAGLE design)
At the start: 5 parts, among them U1 AGND, U2 AGND, U3 AGND

Commit message: commit and push eagle files for Nexus v2.3
Parts:
- removed U1, U2, U3: AGND, CYCFI_Jack:NSJ12HC
- added J1, J2, J3: (no value), CYCFI_Jack:ZHEJINAG_CK_STSJACKS
Connections:
- removed net AGND: H2.5, H2.6, H2.7, H2.8, U1G$1.S, U1G$2.S, U1G$3.DGND, U2G$1.S, U2G$2.S, U2G$3.DGND, U3G$1.S, U3G$2.S, U3G$3.DGND
- removed net N$2: H1.2, U1G$1.R
- new net GND: H2.5, H2.6, H2.7, H2.8, J1G$1.S, J1G$2.S, J2G$1.S, J2G$2.S, J3G$1.S, J3G$2.S
- new net N$13: H1.2, J1G$1.R
- net N$1: now also J1G$1.T; no longer U1G$1.T
- net N$10: now also J3G$1.R; no longer U3G$1.R
- net N$11: now also J3G$2.T; no longer U3G$2.T
- net N$12: now also J3G$2.R; no longer U3G$2.R
- net N$3: now also J1G$2.T; no longer U1G$2.T
- net N$4: now also J1G$2.R; no longer U1G$2.R
- net N$5: now also J2G$1.T; no longer U2G$1.T
- net N$6: now also J2G$1.R; no longer U2G$1.R
- net N$7: now also J2G$2.T; no longer U2G$2.T
- net N$8: now also J2G$2.R; no longer U2G$2.R
- net N$9: now also J3G$1.T; no longer U3G$1.T
Other:
- note added: "CH1/2"
- note added: "CH11/12"
- note added: "CH3/4"
- note added: "CH5/6"
- note added: "CH7/8"
- note added: "CH9/10"
- note added: "I/O Board"
- note added: "I/O Module for Nexus Project by Cycfi Research is licensed under a Creative Commons Attribution-ShareAlike 4.0 International License. Copyright CYCFI Research Inc. 2013-2020"
- note added: "v2.3."
- note removed: "2017025"
- note removed: "I/O Module"
- note removed: "Nexus Project by Cycfi Research is licensed under a Creative Commons Attribution-ShareAlike 4.0 International License. http://creativecommons.org/licenses/by-nc/4.0/ Copyright CYCFI Research Inc. 2013-2018"
- note removed: "v2.0"
- moved on the sheet: H1, H2

Commit message: commit io board changes
Other:
- note added: "J1A"
- note added: "J1B"
- note added: "J2A"
- note added: "J2B"
- note added: "J3A"
- note added: "J3B"
Changed lines of the file:
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@@
 <setting verticaltext="up"/>
 </settings>
-<grid distance="0.1" unitdist="inch" unit="inch" style="lines" multiple="1" display="no" altdistance="0.01" altunitdist="inch" altunit="inch"/>
+<grid distance="0.025" unitdist="inch" unit="inch" style="lines" multiple="1" display="yes" altdistance="0.01" altunitdist="inch" altunit="inch"/>
 <layers>
 <layer number="1" name="Top" color="4" fill="1" visible="no" active="no"/>
@@
 <rectangle x1="214.78875" y1="31.90875" x2="222.91675" y2="31.97225" layer="95"/>
 <rectangle x1="223.48825" y1="31.90875" x2="225.83775" y2="31.97225" layer="95"/>
+<text x="196.215" y="136.525" size="1.778" layer="95">J1A</text>
+<text x="163.195" y="136.525" size="1.778" layer="95">J1B</text>
+<text x="163.195" y="98.425" size="1.778" layer="95">J2B</text>
+<text x="196.215" y="98.425" size="1.778" layer="95">J2A</text>
+<text x="196.215" y="62.865" size="1.778" layer="95">J3A</text>
+<text x="163.195" y="62.865" size="1.778" layer="95">J3B</text>
 </plain>
 <instances>
@@
 <instance part="AGND2" gate="GND" x="134.62" y="93.98"/>
 <instance part="AGND6" gate="GND" x="134.62" y="58.42"/>
-<instance part="J1" gate="G$1" x="177.8" y="147.32" rot="MR180"/>
-<instance part="J1" gate="G$2" x="144.78" y="147.32" rot="MR180"/>
-<instance part="J2" gate="G$1" x="177.8" y="109.22" rot="MR180"/>
-<instance part="J2" gate="G$2" x="144.78" y="109.22" rot="MR180"/>
-<instance part="J3" gate="G$1" x="177.8" y="73.66" rot="MR180"/>
-<instance part="J3" gate="G$2" x="144.78" y="73.66" rot="MR180"/>
+<instance part="J1" gate="G$1" x="177.8" y="147.32" smashed="yes" rot="MR180"/>
+<instance part="J1" gate="G$2" x="144.78" y="147.32" smashed="yes" rot="MR180"/>
+<instance part="J2" gate="G$1" x="177.8" y="109.22" smashed="yes" rot="MR180"/>
+<instance part="J2" gate="G$2" x="144.78" y="109.22" smashed="yes" rot="MR180"/>
+<instance part="J3" gate="G$1" x="177.8" y="73.66" smashed="yes" rot="MR180"/>
+<instance part="J3" gate="G$2" x="144.78" y="73.66" smashed="yes" rot="MR180"/>
 </instances>
 <busses>

Commit message: updates
Other:
- note added: "v2.5"
- note removed: "v2.3."
Changed lines of the file:
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@@
 <setting verticaltext="up"/>
 </settings>
-<grid distance="0.025" unitdist="inch" unit="inch" style="lines" multiple="1" display="yes" altdistance="0.01" altunitdist="inch" altunit="inch"/>
+<grid distance="0.1" unitdist="inch" unit="inch" style="lines" multiple="1" display="no" altdistance="0.01" altunitdist="inch" altunit="inch"/>
 <layers>
 <layer number="1" name="Top" color="4" fill="1" visible="no" active="no"/>
@@
 <plain>
 <text x="203.2" y="19.05" size="2.54" layer="95">I/O Board</text>
-<text x="252.73" y="6.985" size="2.54" layer="95">v2.3.</text>
+<text x="252.73" y="6.985" size="2.54" layer="95">v2.5</text>
 <text x="10.16" y="7.62" size="2.1844" layer="95" font="vector">I/O Module for Nexus Project by Cycfi Research is licensed under a
 Creative Commons Attribution-ShareAlike 4.0 International License.
