File: breakout_box/io_module/io_module.sch (EAGLE design)
At the start: 5 parts, among them U1 AGND, U2 AGND, U3 AGND

Commit message: Update files to version 2.5
Parts:
- removed U1, U2, U3: AGND, CYCFI_Jack:NSJ12HC
- added J1, J2, J3: (no value), CYCFI_Jack:ZHEJINAG_CK_STSJACKS
Connections:
- removed net AGND: H2.5, H2.6, H2.7, H2.8, U1G$1.S, U1G$2.S, U1G$3.DGND, U2G$1.S, U2G$2.S, U2G$3.DGND, U3G$1.S, U3G$2.S, U3G$3.DGND
- removed net N$2: H1.2, U1G$1.R
- new net GND: H2.5, H2.6, H2.7, H2.8, J1G$1.S, J1G$2.S, J2G$1.S, J2G$2.S, J3G$1.S, J3G$2.S
- new net N$13: H1.2, J1G$1.R
- net N$1: now also J1G$1.T; no longer U1G$1.T
- net N$10: now also J3G$1.R; no longer U3G$1.R
- net N$11: now also J3G$2.T; no longer U3G$2.T
- net N$12: now also J3G$2.R; no longer U3G$2.R
- net N$3: now also J1G$2.T; no longer U1G$2.T
- net N$4: now also J1G$2.R; no longer U1G$2.R
- net N$5: now also J2G$1.T; no longer U2G$1.T
- net N$6: now also J2G$1.R; no longer U2G$1.R
- net N$7: now also J2G$2.T; no longer U2G$2.T
- net N$8: now also J2G$2.R; no longer U2G$2.R
- net N$9: now also J3G$1.T; no longer U3G$1.T
Other:
- note added: "CH1/2"
- note added: "CH11/12"
- note added: "CH3/4"
- note added: "CH5/6"
- note added: "CH7/8"
- note added: "CH9/10"
- note added: "I/O Board"
- note added: "I/O Module for Nexus Project by Cycfi Research is licensed under a Creative Commons Attribution-ShareAlike 4.0 International License. Copyright CYCFI Research Inc. 2013-2020"
- note added: "J1A"
- note added: "J1B"
- note added: "J2A"
- note added: "J2B"
- note added: "J3A"
- note added: "J3B"
- note added: "v2.5"
- note removed: "2017025"
- note removed: "I/O Module"
- note removed: "Nexus Project by Cycfi Research is licensed under a Creative Commons Attribution-ShareAlike 4.0 International License. http://creativecommons.org/licenses/by-nc/4.0/ Copyright CYCFI Research Inc. 2013-2018"
- note removed: "v2.0"
- moved on the sheet: H1, H2
