File: breakout_box/io_module/io_module.kicad_sch (KiCad schematic)
At the start: 5 parts, among them J1 ZHEJINAG_CK_STSJACKS, J2 ZHEJINAG_CK_STSJACKS, J3 ZHEJINAG_CK_STSJACKS

Commit message: io_module fab updates; update to latest kicad
Connections:
- net GND renamed AGND
