File: breakout_box/main_board/main_board.sch (EAGLE design)
At the start: 31 parts, among them CN1 19PIN_LEMO, Q1 DMP3099L, Q2 DSS6060

Commit message: Update files to version 2.5
Parts:
- removed C7: 1nF, resistor:C-EUC0402K
- removed D1: FM4004W, CYCFI_diode:FM4007W
- removed H10, H11, H12, H13, H5: (no value), con-lstb:MA03-1_EDITED
- removed H14: MA02-1, con-lstb:MA02-1
- removed H9: (no value), con-lstb:MA08-1
- removed L1: 1mH, inductors:SDR
- removed L2: 82uH, resistor:L-EU
- added H17: (no value), con-lstb:MA08-1
- added JP1, JP10, JP11, JP12, JP13, JP2, JP3, JP4, JP5, JP6, JP7, JP8, JP9: (no value), pinhead-2:PINHD-1X03_2.00
- added R3: 12k, resistor:R-EU_R0603
- added R4: 4.7k, resistor:R-EU_R0402
- C1, C3: value 22uF -> 470uF; device resistor:C-EUC0805 -> resistor:CPOL-EU140CLH-1010
- C4: value 1uF -> 470uF; device resistor:C-EUC0603 -> resistor:CPOL-EU140CLH-1010
- C5: value 10uF -> 1uF
- C6: value 1000uF -> 0.1uF; device resistor:CPOL-EU140CLH-1010 -> resistor:C-EUC0603
- H1, H2: value (none) -> DNP
- H3, H4: device con-lstb:MA03-1_EDITED -> con-lstb:MA08-1
- H6: value (none) -> MA02-1; device con-lstb:MA08-1 -> con-lstb:MA02-1
- Q2: value DSS6060 -> TIP122; device CYCFI_semicon:DSS60601MZ4-13 -> CYCFI_semicon:TIP122
- R1: value 1k -> 220R; device resistor:R-EU_R0402 -> resistor:R-EU_R0603
- R2: value 4.7k -> 220R; device resistor:R-EU_R0402 -> resistor:R-EU_R0603
Connections:
- removed net +AVCC: C4.1, C5.1, C7.1, CN1.16, CN1.17, D1.A, H1.14, H1.15, H9.1, H9.2, Q2.E, R2.1
- removed net +DVCC: C3.1, H1.8, H1.9, H9.5, H9.6, L1.2
- removed net N$20: C2.+, Q2.B, R1.1
- new net N$22: H2.15, JP9.1
- new net N$23: JP11.3, JP8.2
- new net N$31: CN1.3, H17.3, H2.3, H3.3
- new net N$39: CN1.4, H17.4, H2.4, H3.4
- new net N$40: JP12.3, JP7.2
- new net N$41: CN1.6, H17.6, H2.6, H3.6
- new net N$43: H2.8, H3.8, JP2.1
- new net N$44: JP13.3, JP6.2
- new net V_AUX: C1.+, H8.5, H8.6, JP10.1, JP11.1, Q1.S, Q2.C, R1.2
- new net V_OUT: C4.+, C5.1, C6.1, CN1.16, CN1.17, H1.12, H1.13, H1.14, H1.15, H8.1, H8.2, Q2.E, R4.1
- net GND: now also C1.-, C3.-, C4.-, C6.2, H1.20, H1.8, H1.9, H4.5, H4.6, H4.7, H4.8, H6.1, H8.3, H8.4, H8.7, H8.8, JP12.1, JP13.1, R3.1; no longer C1.2, C3.2, C4.2, C6.-, C7.2, H1.12, H1.13, H14.1, H7.5, H7.6, H7.7, H7.8, H9.3, H9.4, H9.7, H9.8
- net N$1: now also CN1.2, H17.2, H2.2, H3.2; no longer H2.13, H3.1
- net N$10: now also JP10.3, JP9.2; no longer CN1.6, H2.6, H6.6
- net N$11: now also H3.7, JP1.1; no longer CN1.7, H6.7
- net N$12: now also CN1.7, JP1.2; no longer CN1.8, H2.8, H6.8
- net N$13: now also H1.1, H7.2, JP3.3; no longer CN1.9, H10.2
- net N$14: now also JP4.2; no longer H11.2
- net N$15: now also JP5.2; no longer H12.2
- net N$16: now also JP13.2; no longer H13.2
- net N$17: now also CN1.9, JP3.2; no longer H2.15, H5.1
- net N$18: now also H4.2, JP4.1; no longer H11.1, H7.2
- net N$19: now also H2.13, JP7.1; no longer C1.1, L1.1, L2.1, Q1.S
- net N$2: now also CN1.1, H17.1, H2.1, H3.1; no longer H14.2, Q1.D
- net N$21: now also H2.14, JP8.1; no longer C6.+, D1.C, L2.2, Q2.C, R1.2
- net N$25: now also R4.2; no longer R2.2
- net N$26: now also H7.4, JP5.3; no longer H12.3, H8.3
- net N$27: now also H7.3, JP4.3; no longer H11.3, H8.2
- net N$28: now also H4.4, JP6.1; no longer H13.1, H7.4
- net N$29: now also H4.3, JP5.1; no longer H12.1, H7.3
- net N$3: now also CN1.8, JP2.2; no longer H2.14, H4.1
- net N$30: now also H7.5, JP6.3; no longer H13.3, H8.4
- net N$32: now also H17.7, H4.1, JP3.1; no longer H10.1, H7.1
- net N$33: now also H7.6, JP7.3; no longer H3.3, H8.5
- net N$34: now also H7.7, JP8.3; no longer H4.3, H8.6
- net N$35: now also H7.8, JP9.3; no longer H5.3, H8.7
- net N$36: now also JP12.2; no longer H3.2
- net N$37: now also JP11.2; no longer H4.2
- net N$38: now also JP10.2; no longer H5.2
- net N$4: now also H6.2, Q1.D; no longer CN1.1, H2.1, H6.1
- net N$5: now also H7.1, JP2.3; no longer CN1.2, H2.2, H6.2
- net N$6: now also C3.+, Q2.B, R2.1, R3.2; no longer CN1.3, H2.3, H6.3
- net N$7: now also H17.8, JP1.3; no longer CN1.4, H2.4, H6.4
- net N$8: now also C2.+, R1.1, R2.2; no longer CN1.5, H2.5, H6.5
- net N$9: now also CN1.5, H17.5, H2.5, H3.5; no longer H1.1, H10.3, H8.1
Other:
- note added: "CH15_GK/CV"
- note added: "CH1_GK"
- note added: "CH2_GK"
- note added: "CH3_GK"
- note added: "CH4_GK"
- note added: "CH5_GK"
- note added: "CH6_GK"
- note added: "CH7_GK/CV"
- note added: "CH8_GK/CV"
- note added: "CH9_SW"
- note added: "CV/ SW"
- note added: "H6"
- note added: "Infinity"
- note added: "MONO_GK"
- note added: "Main Board"
- note added: "Main Board for Nexus Project by Cycfi Research is licensed under a Creative Commons Attribution -ShareAlike 4.0 International License. Copyright CYCFI Research Inc. 2013-2020"
- note added: "Nexus"
- note added: "To GK/MIDI Module"
- note added: "V_AUX"
- note added: "V_OUT"
- note added: "v2.5"
- note removed: "+AVCC"
- note removed: "+DVCC"
- note removed: "2016050"
- note removed: "CV"
- note removed: "Channel Distribution"
- note removed: "Main Board for Nexus Project by Cycfi Research is licensed under a Creative Commons Attribution-ShareAlike 4.0 International License. Copyright CYCFI Research Inc. 2013-2016"
- note removed: "Main Power Source"
- note removed: "NC"
- note removed: "NOTE: *CH9_A = Channel9 Audio *CH9_CV = Channel9 Control Voltage *NC = No Connection"
- note removed: "NOTE: *DGND = Digital Ground *AGND = Analog Ground *+12V_REG = 12V Regulated Power Supply"
- note removed: "NOTES: *+12V_REG = 12V Regulater Power Supply for Analog * +12_VREGD = 12V Regulater Power Supply for Digital *AGND = Analog Ground *DGND= Digital Ground"
- note removed: "To MIDI Module"
- note removed: "v0.96"

Commit message: update schematics
Changed lines of the file:
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@@
 <text x="36.83" y="203.835" size="1.778" layer="95" rot="MR0">CH14</text>
 <text x="36.83" y="201.295" size="1.778" layer="95" rot="MR0">CH15</text>
-<text x="30.48" y="198.755" size="1.778" layer="125">V_OUT</text>
-<text x="30.48" y="196.215" size="1.778" layer="125">V_OUT</text>
+<text x="28.575" y="198.755" size="1.778" layer="125">V_OUT</text>
+<text x="28.575" y="196.215" size="1.778" layer="125">V_OUT</text>
 <text x="162.56" y="127" size="1.778" layer="95">A</text>
 <text x="162.56" y="111.76" size="1.778" layer="95">A</text>
@@
 <text x="210.185" y="153.035" size="1.778" layer="95">AGND</text>
 <text x="210.185" y="150.495" size="1.778" layer="95">AGND</text>
-<text x="30.48" y="193.04" size="1.778" layer="95">AGND</text>
-<text x="30.48" y="189.865" size="1.778" layer="95">AGND</text>
+<text x="28.575" y="193.04" size="1.778" layer="95">AGND</text>
+<text x="28.575" y="190.5" size="1.778" layer="95">AGND</text>
 <text x="363.855" y="158.75" size="1.778" layer="95">AGND</text>
 <text x="363.855" y="156.21" size="1.778" layer="95">AGND</text>

Commit message: update main board files
Connections:
- net GND: now also H1.12; no longer H1.16, H1.8, H1.9
- net N$13: now also H1.3; no longer H1.1
- net N$26: now also H1.5; no longer H1.3
- net N$27: now also H1.4; no longer H1.2
- net N$30: now also H1.6; no longer H1.4
- net N$33: now also H1.7; no longer H1.5
- net N$34: now also H1.8; no longer H1.6
- net N$35: now also H1.9; no longer H1.7
- net N$5: now also H1.2
- net N$7: now also H1.1
- net V_OUT: now also H1.16; no longer H1.12
Other:
- note added: "CH10_CV/ GK"
- note added: "CH7_SW"
- note added: "CH8_SW"
- note removed: "CH15_GK/CV"
- note removed: "CH7_GK/CV"
- note removed: "CH8_GK/CV"
- note removed: "CH9_CV"
